File: 1ELx_7805/Empty/7805_1ELB.sch (EAGLE design)
At the start: 7 parts, among them IC4 7805TV

Commit message: Cleaned out NETs
Connections:
- removed net GND: C1.-, C2.-, IC4.GND, LED1.C, X1-2.KL, X2-1.KL
- removed net N$1: C1.+, IC4.VI, X1-1.KL
- removed net N$2: LED1.A, R1.1
- removed net VCC: C2.+, IC4.VO, R1.2, X2-2.KL
Changed lines of the file:
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@@
 </busses>
 <nets>
-<net name="N$1" class="0">
-<segment>
-<pinref part="X1" gate="-1" pin="KL"/>
-<wire x1="-238.76" y1="114.3" x2="-236.22" y2="114.3" width="0.1524" layer="91"/>
-<wire x1="-236.22" y1="114.3" x2="-236.22" y2="129.54" width="0.1524" layer="91"/>
-<pinref part="IC4" gate="A1" pin="VI"/>
-<wire x1="-236.22" y1="129.54" x2="-210.82" y2="129.54" width="0.1524" layer="91"/>
-<pinref part="C1" gate="G$1" pin="+"/>
-<wire x1="-210.82" y1="129.54" x2="-200.66" y2="129.54" width="0.1524" layer="91"/>
-<wire x1="-210.82" y1="116.84" x2="-210.82" y2="129.54" width="0.1524" layer="91"/>
-<junction x="-210.82" y="129.54"/>
-</segment>
-</net>
-<net name="VCC" class="0">
-<segment>
-<pinref part="IC4" gate="A1" pin="VO"/>
-<wire x1="-180.34" y1="129.54" x2="-170.18" y2="129.54" width="0.1524" layer="91"/>
-<wire x1="-170.18" y1="129.54" x2="-142.24" y2="129.54" width="0.1524" layer="91"/>
-<wire x1="-142.24" y1="129.54" x2="-132.08" y2="129.54" width="0.1524" layer="91"/>
-<wire x1="-132.08" y1="129.54" x2="-132.08" y2="116.84" width="0.1524" layer="91"/>
-<pinref part="X2" gate="-2" pin="KL"/>
-<wire x1="-132.08" y1="116.84" x2="-114.3" y2="116.84" width="0.1524" layer="91"/>
-<wire x1="-114.3" y1="116.84" x2="-114.3" y2="114.3" width="0.1524" layer="91"/>
-<pinref part="SUPPLY3" gate="G$1" pin="VCC"/>
-<wire x1="-142.24" y1="137.16" x2="-142.24" y2="129.54" width="0.1524" layer="91"/>
-<junction x="-142.24" y="129.54"/>
-<pinref part="C2" gate="G$1" pin="+"/>
-<wire x1="-170.18" y1="116.84" x2="-170.18" y2="129.54" width="0.1524" layer="91"/>
-<pinref part="R1" gate="G$1" pin="2"/>
-<wire x1="-142.24" y1="121.92" x2="-142.24" y2="129.54" width="0.1524" layer="91"/>
-</segment>
-</net>
-<net name="GND" class="0">
-<segment>
-<pinref part="X1" gate="-2" pin="KL"/>
-<wire x1="-238.76" y1="109.22" x2="-236.22" y2="109.22" width="0.1524" layer="91"/>
-<wire x1="-236.22" y1="109.22" x2="-236.22" y2="91.44" width="0.1524" layer="91"/>
-<wire x1="-236.22" y1="91.44" x2="-210.82" y2="91.44" width="0.1524" layer="91"/>
-<wire x1="-210.82" y1="91.44" x2="-190.5" y2="91.44" width="0.1524" layer="91"/>
-<wire x1="-190.5" y1="91.44" x2="-170.18" y2="91.44" width="0.1524" layer="91"/>
-<wire x1="-170.18" y1="91.44" x2="-142.24" y2="91.44" width="0.1524" layer="91"/>
-<wire x1="-142.24" y1="91.44" x2="-121.92" y2="91.44" width="0.1524" layer="91"/>
-<wire x1="-121.92" y1="91.44" x2="-121.92" y2="109.22" width="0.1524" layer="91"/>
-<pinref part="X2" gate="-1" pin="KL"/>
-<wire x1="-121.92" y1="109.22" x2="-114.3" y2="109.22" width="0.1524" layer="91"/>
-<pinref part="LED1" gate="G$1" pin="C"/>
-<wire x1="-142.24" y1="99.06" x2="-142.24" y2="91.44" width="0.1524" layer="91"/>
-<junction x="-142.24" y="91.44"/>
-<pinref part="C1" gate="G$1" pin="-"/>
-<wire x1="-210.82" y1="109.22" x2="-210.82" y2="91.44" width="0.1524" layer="91"/>
-<junction x="-210.82" y="91.44"/>
-<pinref part="IC4" gate="A1" pin="GND"/>
-<wire x1="-190.5" y1="121.92" x2="-190.5" y2="91.44" width="0.1524" layer="91"/>
-<junction x="-190.5" y="91.44"/>
-<pinref part="GND2" gate="1" pin="GND"/>
-<wire x1="-190.5" y1="88.9" x2="-190.5" y2="91.44" width="0.1524" layer="91"/>
-<pinref part="C2" gate="G$1" pin="-"/>
-<wire x1="-170.18" y1="109.22" x2="-170.18" y2="91.44" width="0.1524" layer="91"/>
-<junction x="-170.18" y="91.44"/>
-</segment>
-</net>
-<net name="N$2" class="0">
-<segment>
-<pinref part="LED1" gate="G$1" pin="A"/>
-<pinref part="R1" gate="G$1" pin="1"/>
-<wire x1="-142.24" y1="106.68" x2="-142.24" y2="111.76" width="0.1524" layer="91"/>
-</segment>
-</net>
 </nets>
 </sheet>
